Commit message: gobilda urdf lidar joint and link added

File: Final Project/gobilda/gobilda_ws/src/gobilda_robot/description/urdf/gobilda_description.urdf.xacro (robot description, xacro)
@@ -35,4 +35,22 @@
         izz="${base_mass / 12.0 * (base_width*base_width + base_length*base_length)}"/>
       </inertial> -->
+  </link>
+ <!--Lidar Joint-->
+  <joint name="lidar_sensor" type="fixed">
+    <parent link="base_link"/>
+    <child link="lidar"/>
+    <origin xyz="0, 0, 0.127">
+  </joint>
+  <link name="lidar">
+    <visual>
+      <geometry>
+        <cylinder radius="0.05" length="0.02">
+      </geometry>
+    </visual>
+    <inertial>
+      <mass value="0.1">
+      <origin xyz="0 0 0.127">
+      <inertia ixx="0.01" ixy="0.0" ixz="0.0">
+    </inertial>
   </link>
   <joint name="left_wheel_joint" type="continuous">

Commit message: Updating Description urdf of robot with dimensions

File: Final Project/gobilda/gobilda_ws/src/gobilda_robot/description/urdf/gobilda_description.urdf.xacro (robot description, xacro)
@@ -5,10 +5,10 @@
   <xacro:property name="PI" value="3.1415926535897931"/>
   <xacro:property name="base_mass" value="0.3" /> <!-- arbitrary value for base mass -->
-  <xacro:property name="base_width" value="0.1" />
-  <xacro:property name="base_length" value="0.1" />
-  <xacro:property name="base_height" value="0.05" />
+  <xacro:property name="base_width" value="0.36" />
+  <xacro:property name="base_length" value="0.43" />
+  <xacro:property name="base_height" value="0.1" />
   <xacro:property name="wheel_mass" value="0.3" /> <!-- arbitrary value for wheel mass -->
-  <xacro:property name="wheel_len" value="0.020" />
-  <xacro:property name="wheel_radius" value="0.015" />
+  <xacro:property name="wheel_len" value="0.34" />
+  <xacro:property name="wheel_radius" value="0.0476" />
   <xacro:property name="z_offset" value="-${base_height/2}" /> <!-- Space btw top of beam and the each joint -->
   <!-- Base Link -->
@@ -37,10 +37,10 @@
   </link>
  <!--Lidar Joint-->
-  <joint name="lidar_sensor" type="fixed">
+  <joint name="laser" type="fixed">
     <parent link="base_link"/>
     <child link="lidar"/>
     <origin xyz="0, 0, 0.127">
   </joint>
-  <link name="lidar">
+  <link name="laser">
     <visual>
       <geometry>
